File: PowerSupply/PowerSupply.kicad_pcb (KiCad board)
At the start: 2 copper layers, 23.9 x 41.5 mm, 13 parts, among them J1 Barrel_Jack_Switch, J2 Conn_01x02_Pin, J3 Conn_01x02_Pin, SW1 SW_DPDT_x2, U1 LM7805_TO220, U2 LM317_TO-220

Commit message: added copper fills
Routing:
- net GND: track 69.1 -> 2.79 mm
- added copper zone on B.Cu, net GND
Changed lines of the file:
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@@
   (segment (start 146.502 126.5555) (end 148.463 128.5165) (width 0.25) (layer "B.Cu") (net 1))
   (segment (start 141.477 111.7755) (end 140.896 111.7755) (width 0.25) (layer "F.Cu") (net 2))
-  (segment (start 144.145 118.7015) (end 141.477 116.0335) (width 0.25) (layer "F.Cu") (net 2))
-  (segment (start 134.493 132.1435) (end 135.763 133.4135) (width 0.25) (layer "F.Cu") (net 2))
-  (segment (start 137.038 115.6335) (end 137.038 125.9715) (width 0.25) (layer "F.Cu") (net 2))
-  (segment (start 137.038 125.9715) (end 134.493 128.5165) (width 0.25) (layer "F.Cu") (net 2))
   (segment (start 131.191 134.9325) (end 131.704 134.9325) (width 0.25) (layer "F.Cu") (net 2))
-  (segment (start 134.493 128.5165) (end 134.493 132.1435) (width 0.25) (layer "F.Cu") (net 2))
-  (segment (start 140.896 111.7755) (end 137.038 115.6335) (width 0.25) (layer "F.Cu") (net 2))
-  (segment (start 144.145 118.7015) (end 148.209 118.7015) (width 0.25) (layer "F.Cu") (net 2))
-  (segment (start 141.477 116.0335) (end 141.477 111.7755) (width 0.25) (layer "F.Cu") (net 2))
-  (segment (start 131.704 134.9325) (end 134.493 132.1435) (width 0.25) (layer "F.Cu") (net 2))
-  (segment (start 130.175 114.3835) (end 135.788 114.3835) (width 0.25) (layer "B.Cu") (net 2))
-  (segment (start 137.282 134.9325) (end 135.763 133.4135) (width 0.25) (layer "B.Cu") (net 2))
-  (segment (start 148.971 134.9325) (end 137.282 134.9325) (width 0.25) (layer "B.Cu") (net 2))
-  (segment (start 135.788 114.3835) (end 137.038 115.6335) (width 0.25) (layer "B.Cu") (net 2))
-  (segment (start 146.177 108.7755) (end 143.177 111.7755) (width 0.25) (layer "B.Cu") (net 2))
   (segment (start 143.177 111.7755) (end 141.477 111.7755) (width 0.25) (layer "B.Cu") (net 2))
   (segment (start 148.971 137.4725) (end 145.923 137.4725) (width 0.25) (layer "F.Cu") (net 3))
@@
   (segment (start 145.923 137.4725) (end 144.15 137.4725) (width 0.25) (layer "F.Cu") (net 3))
   (segment (start 144.145 121.2015) (end 137.033 128.3135) (width 0.25) (layer "F.Cu") (net 4))
+  (segment (start 131.191 137.4725) (end 133.477 135.1865) (width 0.25) (layer "F.Cu") (net 4))
   (segment (start 137.033 128.3135) (end 137.033 128.5165) (width 0.25) (layer "F.Cu") (net 4))
+  (segment (start 133.477 132.461) (end 137.033 128.905) (width 0.25) (layer "F.Cu") (net 4))
+  (segment (start 137.033 128.905) (end 137.033 128.5165) (width 0.25) (layer "F.Cu") (net 4))
+  (segment (start 133.477 135.1865) (end 133.477 132.461) (width 0.25) (layer "F.Cu") (net 4))
   (segment (start 130.937 137.4825) (end 131.694 137.4825) (width 0.25) (layer "F.Cu") (net 4))
   (segment (start 137.033 128.5165) (end 137.033 128.8465) (width 0.25) (layer "B.Cu") (net 4))
-  (segment (start 133.477 135.1865) (end 131.191 137.4725) (width 0.25) (layer "B.Cu") (net 4))
-  (segment (start 137.033 128.5165) (end 133.477 132.0725) (width 0.25) (layer "B.Cu") (net 4))
-  (segment (start 133.477 132.0725) (end 133.477 135.1865) (width 0.25) (layer "B.Cu") (net 4))
   (segment (start 134.498 112.5805) (end 134.498 115.6335) (width 0.25) (layer "F.Cu") (net 5))
   (segment (start 138.049 109.0295) (end 134.498 112.5805) (width 0.25) (layer "F.Cu") (net 5))
@@
   (segment (start 143.383 135.6995) (end 135.763 135.6995) (width 0.25) (layer "F.Cu") (net 7))
   (segment (start 143.383 128.5165) (end 143.383 133.4135) (width 0.25) (layer "F.Cu") (net 7))
+  (zone (net 2) (net_name "GND") (layer "B.Cu") (hatch edge 0.5)
+    (connect_pads yes (clearance 0.5))
+    (min_thickness 0.25) (filled_areas_thickness no)
+    (fill yes (thermal_gap 0.5) (thermal_bridge_width 0.5) (island_removal_mode 1) (island_area_min 10))
+    (polygon
+      (pts
+        (xy 151.892 99.568)
+        (xy 128.778 99.568)
+        (xy 128.778 140.208)
+        (xy 151.892 140.208)
+      )
+    )
+  )
 )
